File: electronics/control_board/driver.kicad_sch (KiCad schematic)
At the start: 9 parts, among them J12 Motor1, U3 TB6612FNG

Commit message: Worked on schematic and layout Added logo
Parts:
- C12: renamed from C9; value 50u -> 100u
- J12: value Motor1 -> (none)
- renumbered C7 to C10, C8 to C11, C4 to C6, C5 to C7, C22 to C8, C6 to C9
Other:
- title: (none) -> Motor driver
